Commit message: revised .macro files and implemented working simulation

File: description/base_plate.xacro (robot description, xacro)
@@ -1,4 +1,8 @@
 <?xml version="1.0"?>
-<robot xmlns:xacro="http://www.ros.org/wiki/xacro" >
+<robot xmlns:xacro="http://www.ros.org/wiki/xacro">
+    <!-- user-defined parameters for the base plate -->
+    <xacro:property name="plate_radius" value="0.1143"/>
+    <xacro:property name="plate_length" value="0.005"/>
+    <xacro:property name="plate_mass" value="0.5"/>
     <!-- base plate with user-defined parameters -->
     <xacro:macro name="robot_base_plate" params="parent child xyz rpy">
@@ -13,7 +17,7 @@
             <!-- visual -->
             <visual>
-               <!--<origin xyz="${xyz}"/>-->
+                <origin xyz="${plate_radius} 0 ${plate_length/2}" rpy="0 0 0"/>
                 <geometry>
-                    <cylinder radius="0.1143" length="0.005"/>
+                    <cylinder radius="${plate_radius}" length="${plate_length}"/>
                 </geometry>
                 <material name="orange"/>
@@ -21,20 +25,24 @@
             <!-- collision -->
             <collision>
-                <!--<origin xyz="${xyz}"/>-->
+                <origin xyz="${plate_radius} 0 ${plate_length/2}" rpy="0 0 0"/>
                 <geometry>
-                    <cylinder radius="0.1143" length="0.005"/>
+                    <cylinder radius="${plate_radius}" length="${plate_length}"/>
                 </geometry>
             </collision>
             <!-- inertia -->
             <inertial>
-                <mass value="0.5"/>
-                <inertia ixx="${(1/12) * (0.5) * ((3 * 0.1143 * 0.1143) + (0.005 * 0.005))}"
+                <origin xyz="${plate_radius} 0 ${plate_length/2}" rpy="0 0 0"/>
+                <mass value="${plate_mass}"/>
+                <inertia ixx="${(1/12) * (plate_mass) * ((3 * plate_radius * plate_radius) + (plate_length * plate_length))}"
                         ixy="0.0"
                         ixz="0.0"
-                        iyy="${(1/12) * (0.5) * ((3 * 0.1143 * 0.1143) + (0.005 * 0.005))}"
+                        iyy="${(1/12) * (plate_mass) * ((3 * plate_radius * plate_radius) + (plate_length * plate_length))}"
                         iyz="0.0"
-                        izz="${(1/2) * (0.5) * (0.1143 * 0.1143)}"/>
+                        izz="${(1/2) * (plate_mass) * (plate_radius * plate_radius)}"/>
             </inertial>
         </link>
+        <gazebo reference="${child}">
+            <material>Gazebo/Orange</material>
+        </gazebo>
     </xacro:macro>
 </robot>

File: description/caster_wheel.xacro (robot description, xacro)
@@ -3,16 +3,12 @@
     <!-- user-defined parameters for the wheel -->
     <xacro:property name="wheel_radius" value="0.025"/>
-    <xacro:property name="wheel_length" value="0.02"/>
     <xacro:property name="wheel_mass" value="0.1"/>
-    <xacro:property name="collision_radius" value="0.035"/>
     <!-- wheel with user-defined parameters -->
-    <xacro:macro name="robot_wheel" params="parent child xyz rpy abc">
+    <xacro:macro name="robot_caster_wheel" params="parent child xyz">
         <!-- joint -->
-        <joint name="${parent}_to_${child}_joint" type="continuous">
+        <joint name="${parent}_to_${child}_joint" type="fixed">
             <parent link="${parent}"/>
             <child link="${child}"/>
-            <origin xyz="${xyz}" rpy="${rpy}"/>
-            <axis xyz="${abc}"/>
-            <limit effort="0.05" velocity="10.0"/>
+            <origin xyz="${xyz}" rpy="0 0 0"/>
         </joint>
         <!-- link -->
@@ -22,7 +18,7 @@
                 <origin xyz="0 0 0" rpy="0 0 0"/>
                 <geometry>
-                    <cylinder radius="${wheel_radius}" length="${wheel_length}"/>
+                    <sphere radius="${wheel_radius}"/>
                 </geometry>
-                <material name="blue"/>
+                <material name="green"/>
             </visual>
             <!-- collision -->
@@ -30,5 +26,5 @@
                 <origin xyz="0 0 0" rpy="0 0 0"/>
                 <geometry>
-                    <sphere radius="${collision_radius}"/>
+                    <sphere radius="${wheel_radius}"/>
                 </geometry>
             </collision>
@@ -37,14 +33,16 @@
                 <origin xyz="0 0 0" rpy="0 0 0"/>
                 <mass value="${wheel_mass}"/>
-                <inertia ixx="${(1/12) * (wheel_mass) * ((3 * wheel_radius * wheel_radius) + (wheel_length * wheel_length))}"
+                <inertia ixx="${(2/5) * (wheel_mass) * (wheel_radius * wheel_radius)}"
                         ixy="0.0"
                         ixz="0.0"
-                        iyy="${(1/12) * (wheel_mass) * ((3 * wheel_radius * wheel_radius) + (wheel_length * wheel_length))}"
+                        iyy="${(2/5) * (wheel_mass) * (wheel_radius * wheel_radius)}"
                         iyz="0.0"
-                        izz="${(1/2) * (wheel_mass) * (wheel_radius * wheel_radius)}"/>
+                        izz="${(2/5) * (wheel_mass) * (wheel_radius * wheel_radius)}"/>
             </inertial>
         </link>
         <gazebo reference="${child}">
-            <material>Gazebo/Blue</material>
+            <material>Gazebo/Green</material>
+            <mu1 value="0.001"/>
+            <mu2 value="0.001"/>
         </gazebo>
     </xacro:macro>

File: description/material_colors.xacro (robot description, xacro)
@@ -1,4 +1,4 @@
 <?xml version="1.0"?>
-<robot xmlns:xacro="http://www.ros.org/wiki/xacro" >
+<robot xmlns:xacro="http://www.ros.org/wiki/xacro">
     <!-- Color links -->
     <material name="white">
@@ -15,5 +15,5 @@
     </material>
     <material name="green">
-        <color rgba="0.0 1 0.0 1" />
+        <color rgba="0 1 0 1" />
     </material>
     <material name="grey">

File: description/pillar.xacro (robot description, xacro)
@@ -1,4 +1,8 @@
 <?xml version="1.0"?>
-<robot xmlns:xacro="http://www.ros.org/wiki/xacro" >
+<robot xmlns:xacro="http://www.ros.org/wiki/xacro">
+    <!-- user-defined parameters for the pillar -->
+    <xacro:property name="pillar_radius" value="0.005"/>
+    <xacro:property name="pillar_length" value="0.0508"/>
+    <xacro:property name="pillar_mass" value="0.1"/>
     <!-- pillar with user-defined parameters -->
     <xacro:macro name="robot_pillar" params="parent child xyz rpy">
@@ -13,7 +17,7 @@
             <!-- visual -->
             <visual>
-               <!--<origin xyz="${xyz}"/>-->
+                <origin xyz="0 0 ${pillar_length/2}" rpy="0 0 0"/>
                 <geometry>
-                    <cylinder radius="0.005" length="0.0508"/>
+                    <cylinder radius="${pillar_radius}" length="${pillar_length}"/>
                 </geometry>
                 <material name="white"/>
@@ -21,20 +25,24 @@
             <!-- collision -->
             <collision>
-                <!--<origin xyz="${xyz}"/>-->
+                <origin xyz="0 0 ${pillar_length/2}" rpy="0 0 0"/>
                 <geometry>
-                    <cylinder radius="0.005" length="0.0508"/>
+                    <cylinder radius="${pillar_radius}" length="${pillar_length}"/>
                 </geometry>
             </collision>
             <!-- inertia -->
             <inertial>
-                <mass value="0.1"/>
-                <inertia ixx="${(1/12) * (0.1) * ((3 * 0.1143 * 0.1143) + (0.005 * 0.005))}"
+                <origin xyz="0 0 ${pillar_length/2}" rpy="0 0 0"/>
+                <mass value="${pillar_mass}"/>
+                <inertia ixx="${(1/12) * (pillar_mass) * ((3 * pillar_radius * pillar_radius) + (pillar_length * pillar_length))}"
                         ixy="0.0"
                         ixz="0.0"
-                        iyy="${(1/12) * (0.1) * ((3 * 0.1143 * 0.1143) + (0.005 * 0.005))}"
+                        iyy="${(1/12) * (pillar_mass) * ((3 * pillar_radius * pillar_radius) + (pillar_length * pillar_length))}"
                         iyz="0.0"
-                        izz="${(1/2) * (0.1) * (0.1143 * 0.1143)}"/>
+                        izz="${(1/2) * (pillar_mass) * (pillar_radius * pillar_radius)}"/>
             </inertial>
         </link>
+        <gazebo reference="${child}">
+            <material>Gazebo/White</material>
+        </gazebo>
     </xacro:macro>
 </robot>

File: description/robot_core.xacro (robot description, xacro)
@@ -7,7 +7,7 @@
     <xacro:include filename="pillar.xacro"/>
     <xacro:include filename="drive_wheel.xacro"/>
-    <xacro:include filename="castor_wheel.xacro"/>
-    <!-- world link -->
-    <link name="world_link"/>
+    <xacro:include filename="caster_wheel.xacro"/>
+    <!-- base link -->
+    <link name="base_link"/>
     <!-- base plate layers -->
     <!--
@@ -23,5 +23,5 @@
     <!--
         base plate 0 coordinates:
-            x: 0
+            x: -r = -0.1143
             y: 0
             z: 0.075
@@ -35,5 +35,5 @@
             z: t + p = 0.0558
     -->
-    <xacro:robot_base_plate parent="world_link" child="first_base_plate_link" xyz="0 0 0.075" rpy="0 0 0"/>
+    <xacro:robot_base_plate parent="base_link" child="first_base_plate_link" xyz="-0.1143 0 0.075" rpy="0 0 0"/>
     <xacro:robot_base_plate parent="first_base_plate_link" child="second_base_plate_link" xyz="0 0 0.0558" rpy="0 0 0"/>
     <xacro:robot_base_plate parent="second_base_plate_link" child="third_base_plate_link" xyz="0 0 0.0558" rpy="0 0 0"/>
@@ -46,64 +46,54 @@
     -->
     <!-- pillar offset variables -->
-    <xacro:property name="pillar_z_offset" value="0.0279"/>
-    <xacro:property name="pillar_xy_offset" value="0.0708"/>
-    <xacro:property name="pillar_xy_offset_1" value="0"/>
-    <xacro:property name="pillar_radius_offset" value="0.1001"/>
-    <!-- pillars for base layer 0 -->
-    <!--
-        front-right corner coordinates:
-            x_1: (x + (r / sqrt(2))) - o = 0.0808 - o = 0.0708
-            y_1: (y + (r / sqrt(2))) - o = 0.0808 - o = 0.0708
-            z_1: (t / 2) + (p / 2) = 0.0279
-        front-left corner coordinates:
-            x_2: (x - (r / sqrt(2))) + o = -0.0808 + o = -0.0708
-            y_2: (y + (r / sqrt(2))) - o = 0.0808 - o = 0.0708
-            z_2: (t / 2) + (p / 2) = 0.0279
-        back-right corner coordinates:
-            x_3: (x + (r / sqrt(2))) - o = 0.0808 - o = 0.0708
-            y_3: (y - (r / sqrt(2))) + o = -0.0808 + o = -0.0708
-            z_3: (t / 2) + (p / 2) = 0.0279
-        back-left corner coordinates:
-            x_4: (x - (r / sqrt(2))) + o = -0.0808 + o = -0.0708
-            y_4: (y - (r / sqrt(2))) + o = -0.0808 + o = -0.0708
-            z_4: (t / 2) + (p / 2) = 0.0279
-    -->
-    <xacro:robot_pillar parent="first_base_plate_link" child="first_base_plate_front_right_pillar_link" xyz="${pillar_xy_offset} ${pillar_xy_offset} ${pillar_z_offset}" rpy="0 0 0"/>
-    <xacro:robot_pillar parent="first_base_plate_link" child="first_base_plate_front_left_pillar_link" xyz="${-pillar_xy_offset} ${pillar_xy_offset} ${pillar_z_offset}" rpy="0 0 0"/>
-    <xacro:robot_pillar parent="first_base_plate_link" child="first_base_plate_back_right_pillar_link" xyz="${pillar_xy_offset} ${-pillar_xy_offset} ${pillar_z_offset}" rpy="0 0 0"/>
-    <xacro:robot_pillar parent="first_base_plate_link" child="first_base_plate_back_left_pillar_link" xyz="${-pillar_xy_offset} ${-pillar_xy_offset} ${pillar_z_offset}" rpy="0 0 0"/>
-    <!-- pillars for base layer 1 -->
-    <!--
-        front-right corner coordinates:
-            x_1: (x + (r / sqrt(2))) - o = 0.0808 - o = 0.0708
-            y_1: (y + (r / sqrt(2))) - o = 0.0808 - o = 0.0708
-            z_1: (t / 2) + (p / 2) = 0.0279
-        front-left corner coordinates:
-            x_2: (x - (r / sqrt(2))) + o = -0.0808 + o = -0.0708
-            y_2: (y + (r / sqrt(2))) - o = 0.0808 - o = 0.0708
-            z_2: (t / 2) + (p / 2) = 0.0279
-        back-right corner coordinates:
-            x_3: (x + (r / sqrt(2))) - o = 0.0808 - o = 0.0708
-            y_3: (y - (r / sqrt(2))) + o = -0.0808 + o = -0.0708
-            z_3: (t / 2) + (p / 2) = 0.0279
-        back-left corner coordinates:
-            x_4: (x - (r / sqrt(2))) + o = -0.0808 + o = -0.0708
-            y_4: (y - (r / sqrt(2))) + o = -0.0808 + o = -0.0708
-            z_4: (t / 2) + (p / 2) = 0.0279
-    -->
-    <xacro:robot_pillar parent="second_base_plate_link" child="second_base_plate_front_right_pillar_link" xyz="${pillar_xy_offset} ${pillar_xy_offset} ${pillar_z_offset}" rpy="0 0 0"/>
-    <xacro:robot_pillar parent="second_base_plate_link" child="second_base_plate_front_left_pillar_link" xyz="${-pillar_xy_offset} ${pillar_xy_offset} ${pillar_z_offset}" rpy="0 0 0"/>
-    <xacro:robot_pillar parent="second_base_plate_link" child="second_base_plate_back_right_pillar_link" xyz="${pillar_xy_offset} ${-pillar_xy_offset} ${pillar_z_offset}" rpy="0 0 0"/>
-    <xacro:robot_pillar parent="second_base_plate_link" child="second_base_plate_back_left_pillar_link" xyz="${-pillar_xy_offset} ${-pillar_xy_offset} ${pillar_z_offset}" rpy="0 0 0"/>
-    <!-- this is if you want to have alternate cross diamond patterns
-    <xacro:robot_pillar parent="second_base_plate_link" child="second_base_plate_front_right_pillar_link" xyz="${pillar_xy_offset_1} ${pillar_radius_offset} ${pillar_z_offset}" rpy="0 0 0"/>
-    <xacro:robot_pillar parent="second_base_plate_link" child="second_base_plate_front_left_pillar_link" xyz="${-pillar_radius_offset} ${pillar_xy_offset_1} ${pillar_z_offset}" rpy="0 0 0"/>
-    <xacro:robot_pillar parent="second_base_plate_link" child="second_base_plate_back_right_pillar_link" xyz="${pillar_radius_offset} ${pillar_xy_offset_1} ${pillar_z_offset}" rpy="0 0 0"/>
-    <xacro:robot_pillar parent="second_base_plate_link" child="second_base_plate_back_left_pillar_link" xyz="${pillar_xy_offset_1} ${-pillar_radius_offset} ${pillar_z_offset}" rpy="0 0 0"/>
-    -->
+    <xacro:property name="pillar_x_front" value="0.1851"/>
+    <xacro:property name="pillar_x_back" value="0.0435"/>
+    <xacro:property name="pillar_y_offset" value="0.0708"/>
+    <xacro:property name="pillar_z_offset" value="0.005"/>
+    <!-- pillars for base plate 0 -->
+    <xacro:robot_pillar parent="first_base_plate_link"
+        child="first_base_plate_front_right_pillar_link"
+        xyz="${pillar_x_front} ${pillar_y_offset} ${pillar_z_offset}"
+        rpy="0 0 0"
+    />
+    <xacro:robot_pillar parent="first_base_plate_link"
+        child="first_base_plate_front_left_pillar_link"
+        xyz="${pillar_x_front} ${-pillar_y_offset} ${pillar_z_offset}"
+        rpy="0 0 0"
+    />
+    <xacro:robot_pillar parent="first_base_plate_link"
+        child="first_base_plate_back_right_pillar_link"
+        xyz="${pillar_x_back} ${pillar_y_offset} ${pillar_z_offset}"
+        rpy="0 0 0"
+    />
+    <xacro:robot_pillar parent="first_base_plate_link"
+        child="first_base_plate_back_left_pillar_link"
+        xyz="${pillar_x_back} ${-pillar_y_offset} ${pillar_z_offset}"
+        rpy="0 0 0"
+    />
+    <!-- pillars for base plate 1 -->
+    <xacro:robot_pillar parent="second_base_plate_link"
+        child="second_base_plate_front_right_pillar_link"
+        xyz="${pillar_x_front} ${pillar_y_offset} ${pillar_z_offset}"
+        rpy="0 0 0"
+    />
+    <xacro:robot_pillar parent="second_base_plate_link"
+        child="second_base_plate_front_left_pillar_link"
+        xyz="${pillar_x_front} ${-pillar_y_offset} ${pillar_z_offset}"
+        rpy="0 0 0"
+    />
+    <xacro:robot_pillar parent="second_base_plate_link"
+        child="second_base_plate_back_right_pillar_link"
+        xyz="${pillar_x_back} ${pillar_y_offset} ${pillar_z_offset}"
+        rpy="0 0 0"
+    />
+    <xacro:robot_pillar parent="second_base_plate_link"
+        child="second_base_plate_back_left_pillar_link"
+        xyz="${pillar_x_back} ${-pillar_y_offset} ${pillar_z_offset}"
+        rpy="0 0 0"
+    />
     <!-- drive wheels -->
-    <xacro:robot_wheel parent="first_base_plate_link" child="left_wheel_link" xyz="0 0.124 0" rpy="-${pi/2} 0 0" abc="0 0 1"/>
-    <xacro:robot_wheel parent="first_base_plate_link" child="right_wheel_link" xyz="0 -0.124 0" rpy="${pi/2} 0 0" abc="0 0 -1"/>
-    <!-- castor wheel -->
-     <xacro:robot_castor_wheel parent="first_base_plate_link" child="castor_wheel_link" xyz="0.05 0 0"/>
+    <xacro:robot_wheel parent="base_link" child="left_wheel_link" xyz="0 0.124 0.075" rpy="-${pi/2} 0 0" abc="0 0 1"/>
+    <xacro:robot_wheel parent="base_link" child="right_wheel_link" xyz="0 -0.124 0.075" rpy="${pi/2} 0 0" abc="0 0 -1"/>
+    <!-- caster wheel -->
+    <xacro:robot_caster_wheel parent="first_base_plate_link" child="caster_wheel_link" xyz="0.174 0 0"/>
 </robot>
