Commit message: implemented lidar sensor and temporarily fixed gazebo lidar bug

File: description/base_plate.xacro (robot description, xacro)
@@ -5,11 +5,13 @@
     <xacro:property name="plate_length" value="0.005"/>
     <xacro:property name="plate_mass" value="0.5"/>
+    <xacro:property name="I_plate" value="${(1/12) * (plate_mass) * ((3 * plate_radius * plate_radius) + (plate_length * plate_length))}"/>
+    <xacro:property name="Iz_plate" value="${(1/2) * (plate_mass) * (plate_radius * plate_radius)}"/>
     <!-- base plate with user-defined parameters -->
-    <xacro:macro name="robot_base_plate" params="parent child xyz rpy">
+    <xacro:macro name="robot_base_plate" params="parent child x y z row pitch yaw">
         <!-- joint -->
         <joint name="${child}_joint" type="fixed">
             <parent link="${parent}"/>
             <child link="${child}"/>
-            <origin xyz="${xyz}" rpy="${rpy}"/>
+            <origin xyz="${x} ${y} ${z}" rpy="${row} ${pitch} ${yaw}"/>
         </joint>
         <!-- link -->
@@ -34,10 +36,10 @@
                 <origin xyz="${plate_radius} 0 ${plate_length/2}" rpy="0 0 0"/>
                 <mass value="${plate_mass}"/>
-                <inertia ixx="${(1/12) * (plate_mass) * ((3 * plate_radius * plate_radius) + (plate_length * plate_length))}"
+                <inertia ixx="${I_plate}"
                         ixy="0.0"
                         ixz="0.0"
-                        iyy="${(1/12) * (plate_mass) * ((3 * plate_radius * plate_radius) + (plate_length * plate_length))}"
+                        iyy="${I_plate}"
                         iyz="0.0"
-                        izz="${(1/2) * (plate_mass) * (plate_radius * plate_radius)}"/>
+                        izz="${Iz_plate}"/>
             </inertial>
         </link>

File: description/caster_wheel.xacro (robot description, xacro)
@@ -4,11 +4,12 @@
     <xacro:property name="wheel_radius" value="0.025"/>
     <xacro:property name="wheel_mass" value="0.1"/>
+    <xacro:property name="I_wheel" value="${(2/5) * (wheel_mass) * (wheel_radius * wheel_radius)}"/>
     <!-- wheel with user-defined parameters -->
-    <xacro:macro name="robot_caster_wheel" params="parent child xyz">
+    <xacro:macro name="robot_caster_wheel" params="parent child x y z">
         <!-- joint -->
         <joint name="${parent}_to_${child}_joint" type="fixed">
             <parent link="${parent}"/>
             <child link="${child}"/>
-            <origin xyz="${xyz}" rpy="0 0 0"/>
+            <origin xyz="${x} ${y} ${z}" rpy="0 0 0"/>
         </joint>
         <!-- link -->
@@ -33,10 +34,10 @@
                 <origin xyz="0 0 0" rpy="0 0 0"/>
                 <mass value="${wheel_mass}"/>
-                <inertia ixx="${(2/5) * (wheel_mass) * (wheel_radius * wheel_radius)}"
+                <inertia ixx="${I_wheel}"
                         ixy="0.0"
                         ixz="0.0"
-                        iyy="${(2/5) * (wheel_mass) * (wheel_radius * wheel_radius)}"
+                        iyy="${I_wheel}"
                         iyz="0.0"
-                        izz="${(2/5) * (wheel_mass) * (wheel_radius * wheel_radius)}"/>
+                        izz="${I_wheel}"/>
             </inertial>
         </link>

File: description/drive_wheel.xacro (robot description, xacro)
@@ -5,13 +5,15 @@
     <xacro:property name="wheel_length" value="0.02"/>
     <xacro:property name="wheel_mass" value="0.1"/>
-    <xacro:property name="collision_radius" value="0.035"/>
+    <xacro:property name="collision_radius" value="0.025"/>
+    <xacro:property name="I_wheel" value="${(1/12) * (wheel_mass) * ((3 * wheel_radius * wheel_radius) + (wheel_length * wheel_length))}"/>
+    <xacro:property name="Iz_wheel" value="${(1/2) * (wheel_mass) * (wheel_radius * wheel_radius)}"/>
     <!-- wheel with user-defined parameters -->
-    <xacro:macro name="robot_wheel" params="parent child xyz rpy abc">
+    <xacro:macro name="robot_wheel" params="parent child x y z row pitch yaw a b c">
         <!-- joint -->
         <joint name="${parent}_to_${child}_joint" type="continuous">
             <parent link="${parent}"/>
             <child link="${child}"/>
-            <origin xyz="${xyz}" rpy="${rpy}"/>
-            <axis xyz="${abc}"/>
+            <origin xyz="${x} ${y} ${z}" rpy="${row} ${pitch} ${yaw}"/>
+            <axis xyz="${a} ${b} ${c}"/>
             <limit effort="0.05" velocity="10.0"/>
         </joint>
@@ -37,10 +39,10 @@
                 <origin xyz="0 0 0" rpy="0 0 0"/>
                 <mass value="${wheel_mass}"/>
-                <inertia ixx="${(1/12) * (wheel_mass) * ((3 * wheel_radius * wheel_radius) + (wheel_length * wheel_length))}"
+                <inertia ixx="${I_wheel}"
                         ixy="0.0"
                         ixz="0.0"
-                        iyy="${(1/12) * (wheel_mass) * ((3 * wheel_radius * wheel_radius) + (wheel_length * wheel_length))}"
+                        iyy="${I_wheel}"
                         iyz="0.0"
-                        izz="${(1/2) * (wheel_mass) * (wheel_radius * wheel_radius)}"/>
+                        izz="${Iz_wheel}"/>
             </inertial>
         </link>

File: description/gazebo_control.xacro (robot description, xacro)
@@ -1,4 +1,9 @@
 <?xml version="1.0"?>
 <robot xmlns:xacro="http://www.ros.org/wiki/xacro">
+    <!--
+        ##################################################
+            Controller for the robot
+        ##################################################
+    -->
     <gazebo>
         <plugin name="gz::sim::systems::DiffDrive" filename="gz-sim-diff-drive-system">
@@ -8,12 +13,21 @@
             <wheel_separation>0.248</wheel_separation>
             <wheel_radius>0.025</wheel_radius>
+            <!-- speed limits -->
+            <max_wheel_torque>200</max_wheel_torque>
+            <max_wheel_acceleration>10.0</max_wheel_acceleration>
             <!-- input -->
             <topic>cmd_vel</topic>
             <!-- output -->
+            <tf_topic>/tf</tf_topic>
+            <odom_topic>odom</odom_topic>
             <frame_id>odom</frame_id>
             <child_frame_id>base_link</child_frame_id>
-            <odom_topic>odom</odom_topic>
-            <tf_topic>tf</tf_topic>
+            <odom_publisher_frequency>30</odom_publisher_frequency>
         </plugin>
+        <!--
+            ##################################################
+                Joint state publisher
+            ##################################################
+        -->
         <plugin name="gz::sim::systems::JointStatePublisher" filename="gz-sim-joint-state-publisher-system">
             <topic>joint_states</topic>
@@ -21,4 +35,10 @@
             <right_joint>base_link_to_right_wheel_link_joint</right_joint>
         </plugin>
+        <!--
+            ##################################################
+        -->
     </gazebo>
+    <!--
+        ##################################################
+    -->
 </robot>

File: description/material_colors.xacro (robot description, xacro)
@@ -20,3 +20,6 @@
         <color rgba="0.5 0.5 0.5 1" />
     </material>
+    <material name="red">
+        <color rgba="1 0 0 1"/>
+    </material>
 </robot>

File: description/pillar.xacro (robot description, xacro)
@@ -5,11 +5,13 @@
     <xacro:property name="pillar_length" value="0.0508"/>
     <xacro:property name="pillar_mass" value="0.1"/>
+    <xacro:property name="I_pillar" value="${(1/12) * (pillar_mass) * ((3 * pillar_radius * pillar_radius) + (pillar_length * pillar_length))}"/>
+    <xacro:property name="Iz_pillar" value="${(1/2) * (pillar_mass) * (pillar_radius * pillar_radius)}"/>
     <!-- pillar with user-defined parameters -->
-    <xacro:macro name="robot_pillar" params="parent child xyz rpy">
+    <xacro:macro name="robot_pillar" params="parent child x y z row pitch yaw">
         <!-- joint -->
         <joint name="${child}_joint" type="fixed">
             <parent link="${parent}"/>
             <child link="${child}"/>
-            <origin xyz="${xyz}" rpy="${rpy}"/>
+            <origin xyz="${x} ${y} ${z}" rpy="${row} ${pitch} ${yaw}"/>
         </joint>
         <!-- link -->
@@ -34,10 +36,10 @@
                 <origin xyz="0 0 ${pillar_length/2}" rpy="0 0 0"/>
                 <mass value="${pillar_mass}"/>
-                <inertia ixx="${(1/12) * (pillar_mass) * ((3 * pillar_radius * pillar_radius) + (pillar_length * pillar_length))}"
+                <inertia ixx="${I_pillar}"
                         ixy="0.0"
                         ixz="0.0"
-                        iyy="${(1/12) * (pillar_mass) * ((3 * pillar_radius * pillar_radius) + (pillar_length * pillar_length))}"
+                        iyy="${I_pillar}"
                         iyz="0.0"
-                        izz="${(1/2) * (pillar_mass) * (pillar_radius * pillar_radius)}"/>
+                        izz="${Iz_pillar}"/>
             </inertial>
         </link>

File: description/robot.urdf.xacro (robot description, xacro)
@@ -1,5 +1,21 @@
 <?xml version="1.0"?>
-<robot xmlns:xacro="http://www.ros.org/wiki/xacro"  name="robot">
+<robot xmlns:xacro="http://www.ros.org/wiki/xacro"  name="nav_bot">
+    <!-- include other xacro files -->
     <xacro:include filename="robot_core.xacro"/>
     <xacro:include filename="gazebo_control.xacro"/>
+    <xacro:include filename="lidar.xacro"/>
+    <!--
+        ##################################################
+            LIDAR sensor
+        ##################################################
+    -->
+    <xacro:robot_lidar
+        parent="third_base_plate_link"
+        child="laser_frame"
+        x="0.174" y="0" z="0.025"
+        row="0" pitch="0" yaw="0"
+    />
+    <!--
+        ##################################################
+    -->
 </robot>

File: description/robot_core.xacro (robot description, xacro)
@@ -1,4 +1,4 @@
 <?xml version="1.0"?>
-<robot xmlns:xacro="http://www.ros.org/wiki/xacro" >
+<robot xmlns:xacro="http://www.ros.org/wiki/xacro">
     <!-- include other xacro files -->
     <xacro:include filename="material_colors.xacro"/>
@@ -8,92 +8,197 @@
     <xacro:include filename="drive_wheel.xacro"/>
     <xacro:include filename="caster_wheel.xacro"/>
-    <!-- base link -->
+    <!--
+        ##################################################
+            Base Link
+        ##################################################
+    -->
     <link name="base_link"/>
-    <!-- base plate layers -->
-    <!--
-        base plate diameter:
-            d: 0.2286
-        base plate radius:
-            r: 0.1143
-        base plate thickness:
-            t: 0.005
-        square side length:
-            sl: sqrt(2) * (d / 2) = 0.1616
-    -->
-    <!--
-        base plate 0 coordinates:
-            x: -r = -0.1143
-            y: 0
-            z: 0.075
-        base plate 1 coordinates:
-            x: 0
-            y: 0
-            z: t + p = 0.0558
-        base plate 2 coordinates:
-            x: 0
-            y: 0
-            z: t + p = 0.0558
-    -->
-    <xacro:robot_base_plate parent="base_link" child="first_base_plate_link" xyz="-0.1143 0 0.075" rpy="0 0 0"/>
-    <xacro:robot_base_plate parent="first_base_plate_link" child="second_base_plate_link" xyz="0 0 0.0558" rpy="0 0 0"/>
-    <xacro:robot_base_plate parent="second_base_plate_link" child="third_base_plate_link" xyz="0 0 0.0558" rpy="0 0 0"/>
-    <!-- pillars -->
-    <!--
-        pillar length:
-            p: 0.0508
-        pillar xy-position offset:
-            o: 0.01
-    -->
-    <!-- pillar offset variables -->
+    <!--
+        ##################################################
+    -->
+    <!--
+        ##################################################
+            Base Plate Layers
+        ##################################################
+        ##################################################
+            Base Plate diameter:
+                d: 0.2286
+            Base Plate radius:
+                r: 0.1143
+            Base Plate thickness:
+                t: 0.005
+            Square side length:
+                sl: sqrt(2) * (d / 2) = 0.1616
+        ##################################################
+        ##################################################
+            Base Plate 0 coordinates:
+                x: -r = -0.1143
+                y: 0
+                z: 0.075
+            Base Plate 1 coordinates:
+                x: 0
+                y: 0
+                z: t + p = 0.0558
+            Base Plate 2 coordinates:
+                x: 0
+                y: 0
+                z: t + p = 0.0558
+        ##################################################
+    -->
+    <xacro:robot_base_plate
+        parent="base_link"
+        child="first_base_plate_link"
+        x="-0.1143" y="0" z="0.075"
+        row="0" pitch="0" yaw="0"
+    />
+    <xacro:robot_base_plate
+        parent="first_base_plate_link"
+        child="second_base_plate_link"
+        x="0" y="0" z="0.0558"
+        row="0" pitch="0" yaw="0"
+    />
+    <xacro:robot_base_plate
+        parent="second_base_plate_link"
+        child="third_base_plate_link"
+        x="0" y="0" z="0.0558"
+        row="0" pitch="0" yaw="0"
+    />
+    <!--
+        ##################################################
+    -->
+    <!--
+        ##################################################
+            Pillars
+        ##################################################
+        ##################################################
+            Pillar length:
+                p: 0.0508
+            Pillar xy-position offset:
+                o: 0.01
+        ##################################################
+    -->
+    <!--
+        ##################################################
+            Pillar offset variables
+        ##################################################
+    -->
     <xacro:property name="pillar_x_front" value="0.1851"/>
     <xacro:property name="pillar_x_back" value="0.0435"/>
     <xacro:property name="pillar_y_offset" value="0.0708"/>
     <xacro:property name="pillar_z_offset" value="0.005"/>
-    <!-- pillars for base plate 0 -->
-    <xacro:robot_pillar parent="first_base_plate_link"
+    <!--
+        ##################################################
+    -->
+    <!--
+        ##################################################
+            Pillars for Base Plate 0
+        ##################################################
+    -->
+    <xacro:robot_pillar
+        parent="first_base_plate_link"
         child="first_base_plate_front_right_pillar_link"
-        xyz="${pillar_x_front} ${pillar_y_offset} ${pillar_z_offset}"
-        rpy="0 0 0"
-    />
-    <xacro:robot_pillar parent="first_base_plate_link"
+        x="${pillar_x_front}" y="${pillar_y_offset}" z="${pillar_z_offset}"
+        row="0" pitch="0" yaw="0"
+    />
+    <xacro:robot_pillar
+        parent="first_base_plate_link"
         child="first_base_plate_front_left_pillar_link"
-        xyz="${pillar_x_front} ${-pillar_y_offset} ${pillar_z_offset}"
-        rpy="0 0 0"
-    />
-    <xacro:robot_pillar parent="first_base_plate_link"
+        x="${pillar_x_front}" y="${-pillar_y_offset}" z="${pillar_z_offset}"
+        row="0" pitch="0" yaw="0"
+    />
+    <xacro:robot_pillar
+        parent="first_base_plate_link"
         child="first_base_plate_back_right_pillar_link"
-        xyz="${pillar_x_back} ${pillar_y_offset} ${pillar_z_offset}"
-        rpy="0 0 0"
-    />
-    <xacro:robot_pillar parent="first_base_plate_link"
+        x="${pillar_x_back}" y="${pillar_y_offset}" z="${pillar_z_offset}"
+        row="0" pitch="0" yaw="0"
+    />
+    <xacro:robot_pillar
+        parent="first_base_plate_link"
         child="first_base_plate_back_left_pillar_link"
-        xyz="${pillar_x_back} ${-pillar_y_offset} ${pillar_z_offset}"
-        rpy="0 0 0"
-    />
-    <!-- pillars for base plate 1 -->
-    <xacro:robot_pillar parent="second_base_plate_link"
+        x="${pillar_x_back}" y="${-pillar_y_offset}" z="${pillar_z_offset}"
+        row="0" pitch="0" yaw="0"
+    />
+    <!--
+        ##################################################
+    -->
+    <!--
+        ##################################################
+            Pillars for Base Plate 1
+        ##################################################
+    -->
+    <xacro:robot_pillar
+        parent="second_base_plate_link"
         child="second_base_plate_front_right_pillar_link"
-        xyz="${pillar_x_front} ${pillar_y_offset} ${pillar_z_offset}"
-        rpy="0 0 0"
-    />
-    <xacro:robot_pillar parent="second_base_plate_link"
+        x="${pillar_x_front}" y="${pillar_y_offset}" z="${pillar_z_offset}"
+        row="0" pitch="0" yaw="0"
+    />
+    <xacro:robot_pillar
+        parent="second_base_plate_link"
         child="second_base_plate_front_left_pillar_link"
-        xyz="${pillar_x_front} ${-pillar_y_offset} ${pillar_z_offset}"
-        rpy="0 0 0"
-    />
-    <xacro:robot_pillar parent="second_base_plate_link"
+        x="${pillar_x_front}" y="${-pillar_y_offset}" z="${pillar_z_offset}"
+        row="0" pitch="0" yaw="0"
+    />
+    <xacro:robot_pillar
+        parent="second_base_plate_link"
         child="second_base_plate_back_right_pillar_link"
-        xyz="${pillar_x_back} ${pillar_y_offset} ${pillar_z_offset}"
-        rpy="0 0 0"
-    />
-    <xacro:robot_pillar parent="second_base_plate_link"
+        x="${pillar_x_back}" y="${pillar_y_offset}" z="${pillar_z_offset}"
+        row="0" pitch="0" yaw="0"
+    />
+    <xacro:robot_pillar
+        parent="second_base_plate_link"
         child="second_base_plate_back_left_pillar_link"
-        xyz="${pillar_x_back} ${-pillar_y_offset} ${pillar_z_offset}"
-        rpy="0 0 0"
-    />
-    <!-- drive wheels -->
-    <xacro:robot_wheel parent="base_link" child="left_wheel_link" xyz="0 0.124 0.075" rpy="-${pi/2} 0 0" abc="0 0 1"/>
-    <xacro:robot_wheel parent="base_link" child="right_wheel_link" xyz="0 -0.124 0.075" rpy="${pi/2} 0 0" abc="0 0 -1"/>
-    <!-- caster wheel -->
-    <xacro:robot_caster_wheel parent="first_base_plate_link" child="caster_wheel_link" xyz="0.174 0 0"/>
+        x="${pillar_x_back}" y="${-pillar_y_offset}" z="${pillar_z_offset}"
+        row="0" pitch="0" yaw="0"
+    />
+    <!--
+        ##################################################
+    -->
+    <!--
+        ##################################################
+    -->
+    <!--
+        ##################################################
+            Drive Wheels
+        ##################################################
+    -->
+    <xacro:robot_wheel
+        parent="base_link"
+        child="left_wheel_link"
+        x="0" y="0.124" z="0.075"
+        row="${-pi/2}" pitch="0" yaw="0"
+        a="0" b="0" c="1"
+    />
+    <xacro:robot_wheel
+        parent="base_link"
+        child="right_wheel_link"
+        x="0" y="-0.124" z="0.075"
+        row="${pi/2}" pitch="0" yaw="0"
+        a="0" b="0" c="-1"
+    />
+    <!--
+        ##################################################
+    -->
+    <!--
+        ##################################################
+            Caster Wheels
+        ##################################################
+        ##################################################
+            Front x: 0.174
+            Center: 0.1143
+            Back x: Center - (Front x - Center): 0.0546
+        ##################################################
+    -->
+    <xacro:robot_caster_wheel
+        parent="first_base_plate_link"
+        child="front_caster_wheel_link"
+        x="0.174" y="0" z="0"
+    />
+    <xacro:robot_caster_wheel
+        parent="first_base_plate_link"
+        child="back_caster_wheel_link"
+        x="0.0546" y="0" z="0"
+    />
+    <!--
+        ##################################################
+    -->
 </robot>
