Commit message: implemented SLAM, updated cmd_vel topic, updated robot's velocity, and included another camera sensor

File: description/camera.xacro (robot description, xacro)
@@ -25,5 +25,5 @@
                     <box size="${camera_length} ${camera_width} ${camera_height}"/>
                 </geometry>
-                <material name="red"/>
+                <material name="grey"/>
             </visual>
             <!-- collision -->
@@ -55,5 +55,5 @@
         <link name="${child}_optical"></link>
         <gazebo reference="${child}">
-            <material>Gazebo/Red</material>
+            <material>Gazebo/Grey</material>
             <sensor name="camera" type="camera">
                 <pose relative_to="${child}"> 0 0 0 0 0 0 </pose>

File: description/depth_camera.xacro (robot description, xacro)
@@ -25,5 +25,5 @@
                     <box size="${camera_length} ${camera_width} ${camera_height}"/>
                 </geometry>
-                <material name="red"/>
+                <material name="black"/>
             </visual>
             <!-- collision -->
@@ -50,11 +50,12 @@
             <parent link="${child}"/>
             <child link="${child}_optical"/>
-            <origin xyz="0 0 0" rpy="${-pi/2} 0 ${-pi/2}"/>
+            <!--<origin xyz="0 0 0" rpy="${-pi/2} 0 ${-pi/2}"/>-->
+            <origin xyz="0 0 0" rpy="0 0 0"/>
         </joint>
         <!-- link -->
         <link name="${child}_optical"></link>
         <gazebo reference="${child}">
-            <material>Gazebo/Red</material>
-            <sensor name="camera" type="depth_camera">
+            <material>Gazebo/Black</material>
+            <sensor name="depth_camera" type="depth_camera">
                 <pose relative_to="${child}"> 0 0 0 0 0 0 </pose>
                 <visualize>true</visualize>
@@ -62,5 +63,5 @@
                 <always_on>1</always_on>
                 <camera>
-                    <camera_info_topic>camera/camera_info</camera_info_topic>
+                    <camera_info_topic>depth_camera/camera_info</camera_info_topic>
                     <horizontal_fov>1.089</horizontal_fov>
                     <image>
@@ -74,5 +75,5 @@
                     </clip>
                 </camera>
-                <topic>camera/image_raw</topic>
+                <topic>depth_camera/image_raw</topic>
                 <gz_frame_id>${child}_optical</gz_frame_id>
             </sensor>

File: description/drive_wheel.xacro (robot description, xacro)
@@ -16,5 +16,5 @@
             <origin xyz="${x} ${y} ${z}" rpy="${row} ${pitch} ${yaw}"/>
             <axis xyz="${a} ${b} ${c}"/>
-            <limit effort="0.05" velocity="10.0"/>
+            <limit effort="10.0" velocity="40.0"/>
         </joint>
         <!-- link -->

File: description/lidar.xacro (robot description, xacro)
@@ -65,5 +65,5 @@
                     </range>
                 </lidar>
-                <topic>laser_scanner</topic>
+                <topic>scan</topic>
                 <gz_frame_id>${child}</gz_frame_id>
             </sensor>

File: description/robot.urdf.xacro (robot description, xacro)
@@ -5,5 +5,5 @@
     <xacro:include filename="gazebo_control.xacro"/>
     <xacro:include filename="lidar.xacro"/>
-    <!--<xacro:include filename="camera.xacro"/>-->
+    <xacro:include filename="camera.xacro"/>-
     <xacro:include filename="depth_camera.xacro"/>
     <!--
@@ -23,23 +23,9 @@
     <!--
         ##################################################
-            Camera
+            Camera sensor
         ##################################################
     -->
-    <!--<xacro:robot_camera
-        parent="second_base_plate_link"
-        child="camera_frame"
-        x="0.2186" y="0" z="0.02"
-        row="0" pitch="0" yaw="0"
-    />-->
-    <!--
-        ##################################################
-    -->
-    <!--
-        ##################################################
-            Depth Camera
-        ##################################################
-    -->
-    <xacro:robot_depth_camera
-        parent="second_base_plate_link"
+    <xacro:robot_camera
+        parent="first_base_plate_link"
         child="camera_frame"
         x="0.2186" y="0" z="0.02"
@@ -49,3 +35,17 @@
         ##################################################
     -->
+    <!--
+        ##################################################
+            Depth Camera sensor
+        ##################################################
+    -->
+    <xacro:robot_depth_camera
+        parent="second_base_plate_link"
+        child="camera_depth_frame"
+        x="0.2186" y="0" z="0.02"
+        row="0" pitch="0" yaw="0"
+    />
+    <!--
+        ##################################################
+    -->
 </robot>

File: description/robot_core.xacro (robot description, xacro)
@@ -14,4 +14,18 @@
     -->
     <link name="base_link"/>
+    <!--
+        ##################################################
+    -->
+    <!--
+        ##################################################
+            Base Footprint Link
+        ##################################################
+    -->
+    <joint name="base_footprint_joint" type="fixed">
+        <parent link="base_link"/>
+        <child link="base_footprint"/>
+        <origin xyz="0 0 0" rpy="0 0 0"/>
+    </joint>
+    <link name="base_footprint"/>
     <!--
         ##################################################
